File: pcb/chocbar.sch (KiCad schematic (older format))
At the start: 129 parts, among them SW1 SW_PUSH, SW10 SW_PUSH, SW11 SW_PUSH, SW12 SW_PUSH, SW13 SW_PUSH, SW14 SW_PUSH, SW15 SW_PUSH, SW16 SW_PUSH, SW17 SW_PUSH, SW18 SW_PUSH, SW19 SW_PUSH, SW2 SW_PUSH, SW20 SW_PUSH, SW21 SW_PUSH, SW22 SW_PUSH, SW23 SW_PUSH, SW24 SW_PUSH, SW25 SW_PUSH, SW26 SW_PUSH, SW27 SW_PUSH, SW28 SW_PUSH, SW29 SW_PUSH, SW3 SW_PUSH, SW30 SW_PUSH, SW31 SW_PUSH, SW32 SW_PUSH, SW33 SW_PUSH, SW34 SW_PUSH, SW35 SW_PUSH, SW36 SW_PUSH, SW37 SW_PUSH, SW38 SW_PUSH, SW39 SW_PUSH, SW4 SW_PUSH, SW40 SW_PUSH, SW41 SW_PUSH, SW42 SW_PUSH, SW5 SW_PUSH, SW6 SW_PUSH, SW7 SW_PUSH, SW8 SW_PUSH, SW9 SW_PUSH, U1 ProMicro

Commit message: improve
Parts:
- removed D31, D32, D33, D34, D35, D36, D37, D41, D42: D, mikamo3:D3_SMD_1side, symbol Device:D
- removed L41, L42: SK6812MINI-E, swanmatch:YS-SK6812MINI-E, symbol mikamo3:SK6812MINI-E
- removed SW31, SW32, SW33, SW34, SW35, SW36, SW37, SW41, SW42: SW_PUSH, mikamo3:Choc_Hotswap_1side, symbol foostan:SW_PUSH
- added D10, D18, D19, D20, D28, D8, D9: D, mikamo3:D3_SMD_1side, symbol Device:D
- added SW10, SW18, SW19, SW20, SW28, SW8, SW9: SW_PUSH, mikamo3:Choc_Hotswap_1side, symbol foostan:SW_PUSH
- OL1: footprint foostan:OLED_1side -> mikamo3:OLED_1side
- SW33: renamed from SW24; footprint mikamo3:Choc_Hotswap_1side -> mikamo3:Choc_Hotswap_1.5u_1side
- SW34: renamed from SW25; footprint mikamo3:Choc_Hotswap_1side -> mikamo3:Choc_Hotswap_1.5u_1side
- SW35: renamed from SW26; footprint mikamo3:Choc_Hotswap_1side -> mikamo3:Choc_Hotswap_1.5u_1side
- SW36: renamed from SW27; footprint mikamo3:Choc_Hotswap_1side -> mikamo3:Choc_Hotswap_1.5u_1side
- renumbered D8 to D11, D9 to D12, D10 to D13, D11 to D14, D12 to D15, D13 to D16, D14 to D17, D15 to D21, D16 to D22, D17 to D23, D18 to D24, D19 to D25, D20 to D26, D21 to D27, D22 to D31, D23 to D32, D24 to D33, D25 to D34, D26 to D35, D27 to D36, D28 to D37, SW8 to SW11, SW9 to SW12, SW10 to SW13, SW11 to SW14, SW12 to SW15, SW13 to SW16, SW14 to SW17, SW15 to SW21, SW16 to SW22, SW17 to SW23, SW18 to SW24, SW19 to SW25, SW20 to SW26, SW21 to SW27, SW22 to SW31, SW23 to SW32, SW28 to SW37
Connections:
- net col0: now also U1.11 (8/B4); no longer SW29.1, U1.20 (F4/A3)
- net col1: now also U1.12 (9/B5); no longer SW30.1, U1.19 (F5/A2)
- net col2: now also U1.20 (F4/A3); no longer SW38.1, U1.18 (F6/A1)
- net col3: now also U1.19 (F5/A2); no longer SW39.1, U1.17 (F7/A0)
- net col4: now also U1.18 (F6/A1); no longer SW40.1, U1.16 (B1/15)
- net col5: now also U1.17 (F7/A0); no longer U1.15 (B3/14)
- net col6: now also U1.16 (B1/15); no longer U1.14 (B2/16)
- net row0: now also D10.1 (K), D8.1 (K), D9.1 (K)
- net row1: now also D18.1 (K), D19.1 (K), D20.1 (K)
- net row2: now also D29.1 (K), D30.1 (K), D28.1 (K)
- net row3: now also D38.1 (K), D39.1 (K), D40.1 (K)
- net col9: now reaches U1.13 (B6/10)
- net col9: now also SW30.1, SW40.1, SW10.1, SW20.1
- removed net row4: D29.1 (K), D30.1 (K), U1.11 (8/B4)
- removed net row5: D38.1 (K), D39.1 (K), D40.1 (K), U1.12 (9/B5)
- new net: D8.2 (A), SW8.2
- new net: D9.2 (A), SW9.2
- new net: D10.2 (A), SW10.2
- new net: D18.2 (A), SW18.2
- new net: D19.2 (A), SW19.2
- new net: D20.2 (A), SW20.2
- new net: D28.2 (A), SW28.2
- new net col7: SW18.1, SW28.1, SW38.1, SW8.1, U1.15 (B3/14)
- new net col8: SW19.1, SW29.1, SW39.1, SW9.1, U1.14 (B2/16)
- no-connect marks 4 -> 3
Other:
- moved on the sheet: L1, L10, L11, L12, L13, L14, L15, L16, L17, L18, L19, L2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
